File: Ethernet_Dev_Board/W5500_Dev.kicad_sch (KiCad schematic)
At the start: 30 parts, among them Q1 PMV48XPA2R, U1 WIZNET_W5500, U2 74AUP1T08GWH

Commit message: Added in ESP circuit
Connections:
- net LNKLED: no longer names the net of Q1.1 (G), U1.25 (LINKED)
Changed lines of the file:
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@@
 	)
 	(junction
-		(at 71.126 94.621)
-		(diameter 0)
-		(color 0 0 0 0)
-	)
-	(junction
 		(at 220.345 130.175)
 		(diameter 0)
@@
 	(wire
 		(pts
-			(xy 74.936 94.621) (xy 71.126 94.621)
-		)
-		(stroke
-			(width 0.25)
-			(type solid)
-		)
-	)
-	(wire
-		(pts
 			(xy 29.216 122.561) (xy 37.471 122.561)
 		)
@@
 					(unit 1)
 				)
-			)
-		)
-	)
-	(symbol
-		(lib_id "LED_Controller_Hardware-eagle-import:LNKLED")
-		(at 77.476 94.621 0)
-		(unit 1)
-		(exclude_from_sim no)
-		(in_bom yes)
-		(on_board yes)
-		(dnp no)
-		(property "Reference" "#NetPort012"
-			(at 77.476 94.621 0)
-			(effects
-				(font
-					(size 1.27 1.27)
-				)
-				(hide yes)
-			)
-		)
-		(property "Value" "LNKLED"
-			(at 82.556 94.621 0)
-			(effects
-				(font
-					(size 1.27 1.27)
-				)
-			)
-		)
-		(property "Footprint" ""
-			(at 77.476 94.621 0)
-			(effects
-				(font
-					(size 1.27 1.27)
-				)
-				(hide yes)
-			)
-		)
-		(property "Datasheet" ""
-			(at 77.476 94.621 0)
-			(effects
-				(font
-					(size 1.27 1.27)
-				)
-				(hide yes)
-			)
-		)
-		(property "Description" ""
-			(at 77.476 94.621 0)
-			(effects
-				(font
-					(size 1.27 1.27)
-				)
-				(hide yes)
-			)
-		)
-		(property "Mfg." ""
-			(at 77.476 94.621 0)
-			(effects
-				(font
-					(size 1.27 1.27)
-				)
-				(hide yes)
-			)
-		)
-		(property "Mfg. PN" ""
-			(at 77.476 94.621 0)
-			(effects
-				(font
-					(size 1.27 1.27)
-				)
-				(hide yes)
-			)
-		)
-		(property "Distributor" ""
-			(at 77.476 94.621 0)
-			(effects
-				(font
-					(size 1.27 1.27)
-				)
-				(hide yes)
-			)
-		)
-		(property "Distributor PN" ""
-			(at 77.476 94.621 0)
-			(effects
-				(font
-					(size 1.27 1.27)
-				)
-				(hide yes)
-			)
-		)
-		(pin "1"
-		)
-		(instances
-			(project "Ethernet_Dev_Board"
-				(path "/79118fbd-6cbf-48b1-af39-9f7b00f17642/b5f870de-bc6a-4a5b-89f3-9d8a1777ee09"
-					(reference "#NetPort012")
-					(unit 1)
-				)

Commit message: Added additional oscillator circuit. Re-annotated schematic
Parts:
- added C205: 0.1uF, RG_Capacitors_SMD:0603, symbol LED_Controller_Hardware-eagle-import:CAP-0603
- added R206: 10k, RG_Resistors_SMD:0603, symbol LED_Controller_Hardware-eagle-import:RES-0603
- added R212, R214: 0, RG_Resistors_SMD:0603, symbol RG_resistors:RES-0603
- added Y201: 25MHz, symbol RG_Oscillator:FNETHE
- renumbered C1 to C201, C2 to C202, C4 to C203, C3 to C204, C5 to C206, C9 to C207, C8 to C208, C10 to C209, C11 to C210, D1 to D201, LED1 to LED201, Q1 to Q201, R1 to R201, R2 to R202, R3 to R203, R4 to R204, R5 to R205, R13 to R207, R6 to R208, R14 to R209, R15 to R210, R7 to R211, R16 to R213, R9 to R215, R17 to R216, R10 to R217, R11 to R218, U1 to U201, U2 to U202, XTAL1 to XTAL201
Connections:
- net +3.3V: now also C205.1, R206.1, Y201.4 (Vdd)
- net GNDS: now also C205.2, Y201.2 (GND)
- net XI1: now also R214.1, Y201.3 (CLK); no longer C210.1, R215.1, XTAL201.1
- net XO1: now also R212.1; no longer C209.1, R215.2, XTAL201.3 (3@1)
- new net: C209.1, R212.2, R215.2, XTAL201.3 (3@1)
- new net: R206.2, Y201.1 (OE)
- new net: C210.1, R214.2, R215.1, XTAL201.1
Other:
- moved on the sheet: C203, C209, C210, R215, U202B, XTAL201
